File: KiCad/anemometer/anemometer.kicad_pcb (KiCad board)
At the start: 2 copper layers, 52 x 26 mm, 34 parts, among them U1 LM324, U2 LM393

Commit message: Board Rev 2
Parts:
- removed the R14 at (112.0, 85.0)
- removed the R5 at (116.5, 99.0)
- renumbered C5 to C1, C6 to C2, C2 to C3, C1 to C4, C4 to C5, C3 to C6, R15 to R1, R13 to R10, R17 to R12, R12 to R13, R9 to R14, R10 to R15, R18 to R16, R16 to R2, R1 to R3, R2 to R5, R3 to R6, R6 to R7, R7 to R8, R8 to R9
Routing:
- net Out1: track 24.1 -> 14.0 mm
- net Out2: track 17.8 -> 12.6 mm
- net GND: vias 40 -> 34
Other:
- board text added: "For 3 Stage Amp populate R12 + R16, cut S2_EN 1/2 and solder 2/3"
- board text added: "Rev 2"
- board text removed: "For 3 Stage Amp populate R17 + R18, cut S2_EN 1/2 and solder 2/3"
- board text removed: "Rev 1"
