File: KiCad/anemometer/anemometer.kicad_sch (KiCad schematic)
At the start: 33 parts, among them U1 LM324, U2 LM393

Commit message: Board Rev 2
Parts:
- removed R14, R5: 1k, Resistor_SMD:R_0805_2012Metric_Pad1.20x1.40mm_HandSolder, symbol Device:R
- renumbered C5 to C1, C6 to C2, C2 to C3, C1 to C4, C4 to C5, C3 to C6, R15 to R1, R13 to R10, R17 to R12, R12 to R13, R9 to R14, R10 to R15, R18 to R16, R16 to R2, R1 to R3, R2 to R5, R3 to R6, R6 to R7, R7 to R8, R8 to R9
